Commit message: Succesful Camera Point Cloud transformation - Recognition of problematic glue cubes through Camera Depth Updated - Texture Updated

File: ros2_ws/src/spraying_pathways/urdf/2d_lidar.urdf.xacro (robot description, xacro)
@@ -39,5 +39,5 @@
             </scan>
             <range>
-              <min>0.1</min>
+              <min>0.05</min>
               <max>1.5</max>
               <resolution>0.01</resolution>

File: ros2_ws/src/spraying_pathways/urdf/depth_camera.urdf.xacro (robot description, xacro)
@@ -21,5 +21,5 @@
       <parent link="${parent_link}"/>
       <child link="depth_camera_link"/>
-      <origin xyz="1.0 0.35 1.2" rpy="0 ${pi/2} 0"/>
+      <origin xyz="0.75 0.2 1.0" rpy="0 ${pi/2} 0"/>
     </joint>
     <xacro:if value="${sim_gazebo}">
