Commit message: Safety stop, spraying path with curves & code refactor(add include)

File: ros2_ws/src/spraying_pathways/urdf/depth_camera.urdf.xacro (robot description, xacro)
@@ -21,5 +21,5 @@
       <parent link="${parent_link}"/>
       <child link="depth_camera_link"/>
-      <origin xyz="0.75 0.2 1.0" rpy="0 ${pi/2} 0"/>
+      <origin xyz="2.3 -1.0 2.0" rpy="${pi} ${3*pi/4} ${-pi/6}"/>
     </joint>
     <xacro:if value="${sim_gazebo}">

File: ros2_ws/src/spraying_pathways/urdf/my_robot.urdf.xacro (robot description, xacro)
@@ -16,7 +16,9 @@
   <xacro:include filename="$(find ur_description)/urdf/ur.urdf.xacro" />
   <xacro:include filename="$(find spraying_pathways)/urdf/depth_camera.urdf.xacro" />
+  <xacro:include filename="$(find spraying_pathways)/urdf/depth_camera_ee.urdf.xacro" />
   <xacro:include filename="$(find spraying_pathways)/urdf/2d_lidar.urdf.xacro" />
   <!-- Custom sensors -->
   <xacro:depth_camera parent_link="$(arg tf_prefix)base_link" sim_gazebo="$(arg sim_gazebo)" />
+  <xacro:depth_camera_ee parent_link="$(arg tf_prefix)wrist_3_link" sim_gazebo="$(arg sim_gazebo)" />
   <xacro:lidar_sensor parent_link="$(arg tf_prefix)tool0" tf_prefix="$(arg tf_prefix)" sim_gazebo="$(arg sim_gazebo)" />
 </robot>
